File: mpio_projekty/resetUSBv4.6/resetUSB.kicad_pcb (KiCad board)
At the start: 2 copper layers, 39 x 180 mm, 58 parts, among them J1 USBB-G-SMD, J10 FC68391, J2 TUEA4F2SOBHT, J3 Conn_02x05, J4 SWD_4pin, J5 Conn_02x05, J6 Conn_02x05, J7 AC3MAH-AU-PRE, J8 Mini-Fit Jr; 4,2mm, J9 FC68391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

Commit message: resetUSBv4.8
Parts:
- moved J1 1.00 mm to (117.0, 126.9)
Routing:
- net /RZUTNIK_DP: track 74.4 -> 76.4 mm
- net /RZUTNIK_DM: track 75.7 -> 77.2 mm
- net /RZUTNIK_VBUS: track 78.4 -> 79.4 mm
Changed lines of the file:
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@@
     (thickness 1.6)
     (drawings 24)
-    (tracks 538)
+    (tracks 539)
     (zones 0)
     (modules 58)
@@
   )
   (module mpio:USB-B_SMD (layer F.Cu)
-    (at 117.0375 125.9325 270)
+    (at 117.0375 126.9325 270)
     (descr https://pl.ninigi.com/product/ninigi/gniazdo/usbb-g-smd)
     (tags USBB-G-SMD)
@@
   (gr_line (start 138.1345 88.006) (end 137.3725 88.006) (layer F.SilkS) (width 0.2))
   (gr_line (start 112.0375 175.9325) (end 112.0375 123.9325) (layer F.CrtYd) (width 0.2))
-  (via (at 126.5555 126.5505) (size 1.3) (drill 0.5) (layers F.Cu B.Cu) (net 1))
-  (segment (start 126.5485 126.5575) (end 126.5555 126.5505) (width 0.3) (layer F.Cu) (net 1))
-  (segment (start 124.0375 126.5575) (end 126.5485 126.5575) (width 0.3) (layer F.Cu) (net 1) (status 10))
+  (via (at 126.5555 127.5505) (size 1.3) (drill 0.5) (layers F.Cu B.Cu) (net 1))
+  (segment (start 124.0375 127.5575) (end 126.5485 127.5575) (width 0.3) (layer F.Cu) (net 1) (status 10))
   (segment (start 148.8935 77.2835) (end 148.8935 81.1485) (width 0.3) (layer F.Cu) (net 1) (status 10))
   (segment (start 148.8935 81.1485) (end 148.9075 81.1625) (width 0.3) (layer F.Cu) (net 1))
@@
   (segment (start 114.4905 82.3055) (end 118.6815 86.4965) (width 0.25) (layer F.Cu) (net 18))
   (segment (start 114.4905 69.2245) (end 114.4905 82.3055) (width 0.25) (layer F.Cu) (net 18))
-  (segment (start 126.741502 127.8075) (end 124.0375 127.8075) (width 0.25) (layer F.Cu) (net 18) (status 20))
+  (segment (start 120.4595 66.8115) (end 116.9035 66.8115) (width 0.25) (layer F.Cu) (net 18))
+  (segment (start 127.530501 121.291501) (end 127.530501 128.018501) (width 0.25) (layer F.Cu) (net 18))
   (segment (start 116.9035 66.8115) (end 114.4905 69.2245) (width 0.25) (layer F.Cu) (net 18))
   (segment (start 120.930272 67.282272) (end 120.4595 66.8115) (width 0.25) (layer F.Cu) (net 18))
-  (segment (start 120.4595 66.8115) (end 116.9035 66.8115) (width 0.25) (layer F.Cu) (net 18))
-  (segment (start 120.930272 71.023643) (end 120.930272 67.282272) (width 0.25) (layer F.Cu) (net 18) (status 10))
+  (segment (start 125.7875 128.8075) (end 124.0375 128.8075) (width 0.25) (layer F.Cu) (net 18))
+  (segment (start 120.930272 71.023643) (end 120.930272 67.282272) (width 0.25) (layer F.Cu) (net 18))
   (segment (start 118.6815 86.4965) (end 118.6815 112.4425) (width 0.25) (layer F.Cu) (net 18))
+  (segment (start 126.741502 128.8075) (end 125.7875 128.8075) (width 0.25) (layer F.Cu) (net 18))
   (segment (start 118.6815 112.4425) (end 127.530501 121.291501) (width 0.25) (layer F.Cu) (net 18))
-  (segment (start 127.530501 121.291501) (end 127.530501 127.018501) (width 0.25) (layer F.Cu) (net 18))
-  (segment (start 127.530501 127.018501) (end 126.741502 127.8075) (width 0.25) (layer F.Cu) (net 18))
+  (segment (start 127.530501 128.018501) (end 126.741502 128.8075) (width 0.25) (layer F.Cu) (net 18))
   (segment (start 113.4745 82.8135) (end 117.6655 87.0045) (width 0.25) (layer F.Cu) (net 19))
   (segment (start 113.4745 68.7165) (end 113.4745 82.8135) (width 0.25) (layer F.Cu) (net 19))
   (segment (start 116.279522 65.911478) (end 113.4745 68.7165) (width 0.25) (layer F.Cu) (net 19))
   (segment (start 120.8323 65.911478) (end 116.279522 65.911478) (width 0.25) (layer F.Cu) (net 19))
-  (segment (start 122.530272 67.60945) (end 120.8323 65.911478) (width 0.25) (layer F.Cu) (net 19))
-  (segment (start 122.530272 71.023643) (end 122.530272 67.60945) (width 0.25) (layer F.Cu) (net 19) (status 10))
-  (segment (start 117.6655 112.9505) (end 124.4835 119.7685) (width 0.25) (layer F.Cu) (net 19))
+  (segment (start 122.530272 71.023643) (end 122.530272 67.60945) (width 0.25) (layer F.Cu) (net 19))
   (segment (start 117.6655 87.0045) (end 117.6655 112.9505) (width 0.25) (layer F.Cu) (net 19))
-  (segment (start 124.4835 119.7685) (end 124.4835 123.6115) (width 0.25) (layer F.Cu) (net 19))
-  (segment (start 124.4835 123.6115) (end 124.0375 124.0575) (width 0.25) (layer F.Cu) (net 19) (status 20))
-  (segment (start 124.0375 125.3075) (end 125.1875 125.3075) (width 0.25) (layer F.Cu) (net 20) (status 30))
-  (segment (start 118.1735 112.6965) (end 118.1735 86.7505) (width 0.25) (layer F.Cu) (net 20))
-  (segment (start 118.1735 86.7505) (end 113.9825 82.5595) (width 0.25) (layer F.Cu) (net 20))
-  (segment (start 126.0475 120.5705) (end 118.1735 112.6965) (width 0.25) (layer F.Cu) (net 20))
-  (segment (start 126.0475 124.4475) (end 126.0475 120.5705) (width 0.25) (layer F.Cu) (net 20))
-  (segment (start 125.1875 125.3075) (end 126.0475 124.4475) (width 0.25) (layer F.Cu) (net 20) (status 10))
-  (segment (start 113.9825 82.5595) (end 113.9825 68.9705) (width 0.25) (layer F.Cu) (net 20))
-  (segment (start 113.9825 68.9705) (end 116.591511 66.361489) (width 0.25) (layer F.Cu) (net 20))
-  (segment (start 116.591511 66.361489) (end 120.6459 66.361489) (width 0.25) (layer F.Cu) (net 20))
-  (segment (start 120.6459 66.361489) (end 121.730272 67.445861) (width 0.25) (layer F.Cu) (net 20))
-  (segment (start 121.730272 67.445861) (end 121.730272 71.023643) (width 0.25) (layer F.Cu) (net 20) (status 20))
+  (segment (start 122.530272 67.60945) (end 120.8323 65.911478) (width 0.25) (layer F.Cu) (net 19))
+  (segment (start 117.6655 112.9505) (end 125.0375 120.3225) (width 0.25) (layer F.Cu) (net 19))
+  (segment (start 125.0375 120.3225) (end 125.0375 124.9325) (width 0.25) (layer F.Cu) (net 19))
+  (segment (start 124.1625 124.9325) (end 124.0375 125.0575) (width 0.25) (layer F.Cu) (net 19))
+  (segment (start 125.0375 124.9325) (end 124.1625 124.9325) (width 0.25) (layer F.Cu) (net 19))
+  (segment (start 113.9825 82.5595) (end 118.1735 86.7505) (width 0.25) (layer F.Cu) (net 20))
+  (segment (start 113.9825 68.9705) (end 113.9825 82.5595) (width 0.25) (layer F.Cu) (net 20))
+  (segment (start 116.591511 66.361489) (end 113.9825 68.9705) (width 0.25) (layer F.Cu) (net 20))
+  (segment (start 120.6459 66.361489) (end 116.591511 66.361489) (width 0.25) (layer F.Cu) (net 20))
+  (segment (start 121.730272 71.023643) (end 121.730272 67.445861) (width 0.25) (layer F.Cu) (net 20))
+  (segment (start 118.1735 112.6965) (end 126.2615 120.7845) (width 0.25) (layer F.Cu) (net 20))
+  (segment (start 121.730272 67.445861) (end 120.6459 66.361489) (width 0.25) (layer F.Cu) (net 20))
+  (segment (start 126.2615 125.7085) (end 125.6625 126.3075) (width 0.25) (layer F.Cu) (net 20))
+  (segment (start 118.1735 86.7505) (end 118.1735 112.6965) (width 0.25) (layer F.Cu) (net 20))
+  (segment (start 126.2615 120.7845) (end 126.2615 125.7085) (width 0.25) (layer F.Cu) (net 20))
+  (segment (start 125.6625 126.3075) (end 124.0375 126.3075) (width 0.25) (layer F.Cu) (net 20))
   (segment (start 143.9015 114.2935) (end 143.9015 110.0935) (width 0.75) (layer F.Cu) (net 29) (status 30))
   (segment (start 124.2535 193.5065) (end 122.4315 193.5065) (width 0.75) (layer F.Cu) (net 30))
