File: mpio_projekty/resetUSBv4.95stabilizator/resetUSB.kicad_pcb (KiCad board)
At the start: 2 copper layers, 40 x 158 mm, 66 parts, among them J1 USBB-G-SMD, J10 FC68391, J2 TUEA4F2SOBHT, J3 Conn_02x05, J4 SWD_4pin, J6 Conn_02x05, J7 AC3MAH-AU-PRE, J8 Mini-Fit Jr; 4,2mm, J9 FC68391, Q1 BC817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

Commit message: resetusb pdf
Routing:
- net GND: track 106.2 -> 110.3 mm, vias 11 -> 13
