File: mpio_projekty/resetUSBv4.95stabilizator/resetUSB.kicad_pcb (KiCad board)
At the start: 2 copper layers, 40 x 158 mm, 66 parts, among them J1 USBB-G-SMD, J10 FC68391, J2 TUEA4F2SOBHT, J3 Conn_02x05, J4 SWD_4pin, J6 Conn_02x05, J7 AC3MAH-AU-PRE, J8 Mini-Fit Jr; 4,2mm, J9 FC68391, Q1 BC817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

Commit message: resetUSBv4.98com2
Parts:
- moved J3 10.5 mm to (117.6, 52.5), turned to 0 degrees
Connections:
- C3 pad 1: +5V -> +5P
- J3 pad 1: (no net) -> +5P
- J3 pad 10: (no net) -> Net-(J2-Pad5)
- J3 pad 3: Net-(J2-Pad2) -> /USB_M
- J3 pad 4: /USB_M -> Net-(J2-Pad2)
- J3 pad 5: Net-(J2-Pad3) -> /USB_P
- J3 pad 6: /USB_P -> Net-(J2-Pad3)
- J3 pad 9: Net-(J2-Pad5) -> (no net)
- U1 pad 3: +5V -> +5P
Routing:
- net +5P: track 0.00 -> 35.5 mm
- net +5V: track 222.7 -> 188.6 mm
- net GND: track 106.2 -> 91.4 mm, vias 11 -> 12
- net Net-(J2-Pad2): track 14.9 -> 27.0 mm
- net Net-(J2-Pad5): track 28.3 -> 18.3 mm
- net /USB_M: track 58.2 -> 63.3 mm
