File: mpio_projekty/resetUSBv4.95stabilizator/resetUSB.sch (KiCad schematic (older format))
At the start: 66 parts, among them J1 USBB-G-SMD, J10 FC68391, J2 TUEA4F2SOBHT, J3 Conn_02x05, J4 SWD_4pin, J6 Conn_02x05, J7 AC3MAH-AU-PRE, J8 Mini-Fit Jr; 4,2mm, J9 FC68391, Q1 BC817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

Commit message: resetUSBv4.98com2
Connections:
- net +5V: no longer C3.1, U1.3 (VI)
- net USB_M: now also J3.3 (Pin_3); no longer J3.4 (Pin_4)
- net USB_P: now also J3.5 (Pin_5); no longer J3.6 (Pin_6)
- net at J2.2 (D-): now also J3.4 (Pin_4); no longer J3.3 (Pin_3)
- net at J2.3 (D+): now also J3.6 (Pin_6); no longer J3.5 (Pin_5)
- net at J2.5 (Shield): now also J3.10 (Pin_10); no longer J3.9 (Pin_9)
- net +5P: now reaches J3.1 (Pin_1)
- net +5P: now also C3.1, U1.3 (VI)
- no-connect marks 21 -> 20
Changed lines of the file:
@@
 L conn:Conn_02x05_Odd_Even J3
 U 1 1 5ACB9A54
-P 1950 3600
-F 0 "J3" H 2000 4017 50  0000 C CNN
-F 1 "Conn_02x05" H 2000 3926 50  0000 C CNN
-F 2 "mpio:IDC10" H 1950 3600 50  0001 C CNN
-F 3 "~" H 1950 3600 50  0001 C CNN
-	1    1950 3600
-	1    0    0    -1
+P 2050 3600
+F 0 "J3" H 2100 4017 50  0000 C CNN
+F 1 "Conn_02x05" H 2100 3926 50  0000 C CNN
+F 2 "mpio:IDC10" H 2050 3600 50  0001 C CNN
+F 3 "~" H 2050 3600 50  0001 C CNN
+	1    2050 3600
+	-1   0    0    -1
 $EndComp
 Text Notes 1650 3400 0    60   ~ 0
@@
 F 3 "" H 2350 1800 50  0001 C CNN
 	1    2350 1800
-	1    0    0    -1
-$EndComp
-$Comp
-L power:+5V #PWR09
-U 1 1 5AB4F539
-P 2350 1550
-F 0 "#PWR09" H 2350 1400 50  0001 C CNN
-F 1 "+5V" H 2350 1690 50  0000 C CNN
-F 2 "" H 2350 1550 50  0001 C CNN
-F 3 "" H 2350 1550 50  0001 C CNN
-	1    2350 1550
 	1    0    0    -1
 $EndComp
@@
 	1850 3300 1850 3000
 Connection ~ 1700 3300
-NoConn ~ 2250 3400
 $Comp
 L power:GND #PWR0101
@@
 $EndComp
 $Comp
-L power:GND #PWR?
+L power:GND #PWR0110
 U 1 1 5B34D6E7
 P 1500 3850
-F 0 "#PWR?" H 1500 3600 50  0001 C CNN
+F 0 "#PWR0110" H 1500 3600 50  0001 C CNN
 F 1 "GND" H 1505 3677 50  0000 C CNN
 F 2 "" H 1500 3850 50  0001 C CNN
@@
 	1750 3700 1500 3700
 Connection ~ 1500 3700
+$Comp
+L power:+5P #PWR0111
+U 1 1 5B375963
+P 2300 3350
+F 0 "#PWR0111" H 2300 3200 50  0001 C CNN
+F 1 "+5P" H 2315 3523 50  0000 C CNN
+F 2 "" H 2300 3350 50  0001 C CNN
+F 3 "" H 2300 3350 50  0001 C CNN
+	1    2300 3350
+	1    0    0    -1
+$EndComp
+Wire Wire Line
+	2250 3400 2300 3400
+Wire Wire Line
+	2300 3400 2300 3350
+$Comp
+L power:+5P #PWR0112
+U 1 1 5B38C78B
+P 2350 1550
+F 0 "#PWR0112" H 2350 1400 50  0001 C CNN
+F 1 "+5P" H 2365 1723 50  0000 C CNN
+F 2 "" H 2350 1550 50  0001 C CNN
+F 3 "" H 2350 1550 50  0001 C CNN
+	1    2350 1550
+	1    0    0    -1
+$EndComp
 $EndSCHEMATC
