File: mpio_projekty/audioTransilTest1/audio/audio.kicad_pcb (KiCad board)
At the start: 2 copper layers, 49 parts, among them J1 USB_B, J2 Mini-Fit Jr; 4,2mm, J3 TUEA4F2SOBHT, J4 Conn_02x05, J5 SWD_4pin, Q1 BC817, Q2 BC817, SW1 TACTM-34N-F, U1 STM32F042K6Tx, U2 AP1509-50SG-13, U3 LD1117S33TR, U4 IRLTS2242, U5 AO4616, U6 AO4616

Commit message: resetUSBv4.98com2
Parts:
- removed the C6 at (106.9, 158.5)
- removed the C7 at (100.8, 158.5)
- removed the D3 at (79.5, 161.5)
- removed D5: GREEN, LEDs:LED_0603
- removed D6: BLUE, LEDs:LED_0603
- removed the J1 at (184.3, 58.7)
- removed the J3 at (206.5, 76.7)
- removed J4: Conn_02x05, mpio:IDC10
- removed the L1 at (88.4, 158.5)
- removed L4: 10u, Inductors_SMD:L_0805
- removed R14: 6K8, Resistors_SMD:R_0603
- removed R15: 33K, Resistors_SMD:R_0603
- removed the R7 at (248.7, 165.1)
- removed the U2 at (89.2, 149.1)
- removed the U4 at (123.7, 160.7)
- added J2: USB_B, mpio:USB_Micro-B, F.Cu at (206.5, 76.7)
- added Q3: BC817, TO_SOT_Packages_SMD:SOT-23, F.Cu at (297.4, 33.8)
- added Q4: BC817, TO_SOT_Packages_SMD:SOT-23, F.Cu at (305.8, 23.9)
- added R11: 10K, Resistors_SMD:R_0603, F.Cu at (310.2, 27.8)
- added R12: 10K, Resistors_SMD:R_0603, F.Cu at (301.9, 34.9)
- added R5: 10K, Resistors_SMD:R_0603, F.Cu at (310.2, 22.8)
- added R6: 10K, Resistors_SMD:R_0603, F.Cu at (304.8, 29.9)
- C4: value 100n -> 330u; footprint Capacitors_SMD:C_0603 -> Capacitors_THT:CP_Radial_D16.0mm_P7.50mm
- C5: value 330u -> 10u; footprint Capacitors_SMD:CP_Elec_8x6.5 -> Capacitors_SMD:CP_Elec_5x5.3
- moved C5 270.0 mm to (298.9, 25.3), turned to 0 degrees
- moved C4 144.9 mm to (282.4, 30.7)
- renumbered C11 to C10, C12 to C11, C13 to C3, C8 to C6, C9 to C7, C3 to C8, C10 to C9, D4 to D3, J2 to J1, J5 to J3, L2 to L1, L3 to L2, R3 to R1, R13 to R10, R6 to R2, R12 to R3, R8 to R4, R9 to R7, R10 to R8, R11 to R9, U3 to U2, U5 to U3, U6 to U4
Connections:
- C3 pad 2: GNDA -> GND
- C4 pad 2: GNDA -> GND
- C5 pad 1: +12V -> +5V
- C5 pad 2: GNDA -> GND
- D1 pad 2: GNDA -> GND
- D2 pad 1: GNDA -> GND
- J1 pad 1: GNDA -> GND
- J1 pad 2: GNDA -> GND
- Q1 pad 2: GNDA -> GND
- Q2 pad 2: GNDA -> GND
- R10 pad 2: /LED_RED -> (no net)
- R8 pad 2: /audio_L -> /audio_1
- R9 pad 2: /audio_R -> /audio_2
- SW1 pad 2: /PRZYCISK -> (no net)
- U1 pad 10: /LED_BLUE -> (no net)
- U1 pad 11: /LED_RED -> (no net)
- U1 pad 13: /audio_L -> /audio_1N
- U1 pad 14: /audio_R -> /audio_2N
- U1 pad 18: (no net) -> /audio_1
- U1 pad 19: /PRZYCISK -> /audio_2
- U1 pad 20: /USB_PWR -> (no net)
- U1 pad 9: /LED_GREEN -> (no net)
- U3 pad 1: GNDA -> GND
- U3 pad 2: Net-(Q1-Pad3) -> Net-(Q3-Pad3)
- U4 pad 1: GNDA -> GND
- U4 pad 2: Net-(Q2-Pad3) -> Net-(Q4-Pad3)
Routing:
- net +5V: track 34.3 -> 0.00 mm
- net Net-(D3-Pad1): track 12.5 -> 0.00 mm
- net Net-(C11-Pad1): track 0.00 -> 12.2 mm
- net Net-(C11-Pad2): track 0.00 -> 9.70 mm
- net Net-(C10-Pad2): track 0.00 -> 5.81 mm
- net Net-(C9-Pad1): track 0.00 -> 5.81 mm
- net Net-(Q2-Pad3): track 5.08 -> 4.06 mm
- net Net-(Q1-Pad3): track 5.08 -> 4.06 mm
