File: mpio_projekty/resetUSBv4.98com2/resetUSB.kicad_pcb (KiCad board)
At the start: 2 copper layers, 45 x 165 mm, 68 parts, among them J1 USBB-G-SMD, J10 FC68391, J2 TUEA4F2SOBHT, J3 Conn_02x05, J4 SWD_4pin, J5 DE09-SL-24, J6 Conn_02x05, J7 AC3MAH-AU-PRE, J8 Mini-Fit Jr; 4,2mm, J9 FC68391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

Commit message: resetUSB4.98
Routing:
- net +12V: track 258.3 -> 257.4 mm
Changed lines of the file:
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@@
   (general
     (thickness 1.6)
-    (drawings 29)
-    (tracks 525)
+    (drawings 31)
+    (tracks 524)
     (zones 0)
     (modules 68)
@@
     )
   )
-  (dimension 13 (width 0.3) (layer F.SilkS)
-    (gr_text "13.000 mm" (at 93.1375 88.4325 270) (layer F.SilkS)
+  (dimension 32.5 (width 0.3) (layer F.SilkS)
+    (gr_text "32.500 mm" (at 27.4375 70.6825 90) (layer F.SilkS)
+      (effects (font (size 1.5 1.5) (thickness 0.3)))
+    )
+    (feature1 (pts (xy 51.0375 54.4325) (xy 28.951079 54.4325)))
+    (feature2 (pts (xy 51.0375 86.9325) (xy 28.951079 86.9325)))
+    (crossbar (pts (xy 29.5375 86.9325) (xy 29.5375 54.4325)))
+    (arrow1a (pts (xy 29.5375 54.4325) (xy 30.123921 55.559004)))
+    (arrow1b (pts (xy 29.5375 54.4325) (xy 28.951079 55.559004)))
+    (arrow2a (pts (xy 29.5375 86.9325) (xy 30.123921 85.805996)))
+    (arrow2b (pts (xy 29.5375 86.9325) (xy 28.951079 85.805996)))
+  )
+  (gr_text 12V (at 79.0375 105.4325 90) (layer F.SilkS)
+    (effects (font (size 1 1) (thickness 0.15)))
+  )
+  (dimension 13 (width 0.3) (layer Dwgs.User)
+    (gr_text "13.000 mm" (at 93.1375 88.4325 270) (layer Dwgs.User)
       (effects (font (size 1.5 1.5) (thickness 0.3)))
     )
@@
     (arrow2b (pts (xy 91.0375 81.9325) (xy 91.623921 83.059004)))
   )
-  (dimension 26 (width 0.3) (layer F.SilkS)
-    (gr_text "26.000 mm" (at 98.6375 94.9325 270) (layer F.SilkS)
+  (dimension 26 (width 0.3) (layer Dwgs.User)
+    (gr_text "26.000 mm" (at 98.6375 94.9325 270) (layer Dwgs.User)
       (effects (font (size 1.5 1.5) (thickness 0.3)))
     )
@@
     (arrow2b (pts (xy 44.0375 209.432499) (xy 45.164004 208.846078)))
   )
-  (dimension 11 (width 0.3) (layer F.SilkS)
-    (gr_text "11.000 mm" (at 33.9375 75.4325 90) (layer F.SilkS)
+  (dimension 11 (width 0.3) (layer Dwgs.User)
+    (gr_text "11.000 mm" (at 33.9375 75.4325 90) (layer Dwgs.User)
       (effects (font (size 1.5 1.5) (thickness 0.3)))
     )
@@
     (arrow2b (pts (xy 36.0375 80.9325) (xy 35.451079 79.805996)))
   )
-  (dimension 11 (width 0.3) (layer F.SilkS)
-    (gr_text "11.000 mm" (at 33.9375 98.4325 90) (layer F.SilkS)
+  (dimension 11 (width 0.3) (layer Dwgs.User)
+    (gr_text "11.000 mm" (at 33.9375 98.4325 90) (layer Dwgs.User)
       (effects (font (size 1.5 1.5) (thickness 0.3)))
     )
@@
     (arrow2b (pts (xy 36.0375 103.9325) (xy 35.451079 102.805996)))
   )
-  (dimension 11 (width 0.3) (layer F.SilkS)
-    (gr_text "11.000 mm" (at 31.9375 135.4325 90) (layer F.SilkS)
+  (dimension 11 (width 0.3) (layer Dwgs.User)
+    (gr_text "11.000 mm" (at 31.9375 135.4325 90) (layer Dwgs.User)
       (effects (font (size 1.5 1.5) (thickness 0.3)))
     )
@@
     (arrow2b (pts (xy 34.0375 140.9325) (xy 33.451079 139.805996)))
   )
-  (dimension 11 (width 0.3) (layer F.SilkS)
-    (gr_text "11.000 mm" (at 31.9375 172.4325 90) (layer F.SilkS)
+  (dimension 11 (width 0.3) (layer Dwgs.User)
+    (gr_text "11.000 mm" (at 31.9375 172.4325 90) (layer Dwgs.User)
       (effects (font (size 1.5 1.5) (thickness 0.3)))
     )
@@
   (segment (start 56.4835 79.1365) (end 57.8255 79.1365) (width 0.3) (layer F.Cu) (net 3) (status 10))
   (segment (start 58.3635 79.6745) (end 62.3255 79.6745) (width 0.3) (layer F.Cu) (net 3) (status 20))
+  (segment (start 52.9035 62.0465) (end 49.3715 62.0465) (width 1.8) (layer B.Cu) (net 4))
+  (segment (start 54.9775 59.9725) (end 52.9035 62.0465) (width 1.8) (layer B.Cu) (net 4))
+  (segment (start 49.3715 62.0465) (end 46.8315 64.5865) (width 1.8) (layer B.Cu) (net 4))
+  (segment (start 46.8315 64.5865) (end 46.8315 94.9845) (width 1.8) (layer B.Cu) (net 4))
+  (segment (start 46.8315 94.9845) (end 52.6635 100.8165) (width 1.8) (layer B.Cu) (net 4))
   (segment (start 74.0095 163.6465) (end 76.5495 161.1065) (width 1.8) (layer B.Cu) (net 4))
   (segment (start 74.0095 165.9325) (end 74.0095 163.6465) (width 1.8) (layer B.Cu) (net 4))
@@
   (segment (start 76.5495 144.3425) (end 74.2635 142.0565) (width 1.8) (layer B.Cu) (net 4))
   (segment (start 74.2635 142.0565) (end 74.2635 133.6745) (width 1.8) (layer B.Cu) (net 4) (status 20))
-  (segment (start 46.8315 63.0625) (end 46.8315 94.5585) (width 1.8) (layer B.Cu) (net 4))
-  (segment (start 52.6635 100.8165) (end 46.8315 94.9845) (width 1.8) (layer B.Cu) (net 4) (status 10))
-  (segment (start 46.8315 94.9845) (end 46.8315 94.5585) (width 1.8) (layer B.Cu) (net 4))
   (segment (start 49.1175 115.3865) (end 49.1175 104.3625) (width 1.8) (layer B.Cu) (net 4))
   (segment (start 55.7215 121.9905) (end 49.1175 115.3865) (width 1.8) (layer B.Cu) (net 4))
@@
   (segment (start 52.3355 99.3005) (end 52.6635 99.6285) (width 0.25) (layer F.Cu) (net 4))
   (segment (start 52.3355 97.8115) (end 52.3355 99.3005) (width 0.25) (layer F.Cu) (net 4) (status 10))
-  (segment (start 52.9035 62.0465) (end 47.8475 62.0465) (width 1.8) (layer B.Cu) (net 4))
-  (segment (start 54.9775 59.9725) (end 52.9035 62.0465) (width 1.8) (layer B.Cu) (net 4) (status 10))
-  (segment (start 47.8475 62.0465) (end 46.8315 63.0625) (width 1.8) (layer B.Cu) (net 4))
   (segment (start 74.2635 123.2605) (end 74.2635 120.5665) (width 0.75) (layer F.Cu) (net 4))
   (segment (start 74.2635 133.6745) (end 74.2635 123.2605) (width 0.75) (layer F.Cu) (net 4) (status 10))
@@
     (connect_pads (clearance 0.508))
     (min_thickness 0.254)
-    (fill yes (arc_segments 16) (thermal_gap 0.508) (thermal_bridge_width 0.508))
+    (fill (arc_segments 16) (thermal_gap 0.508) (thermal_bridge_width 0.508))
     (polygon
       (pts
@@
     (connect_pads (clearance 0.508))
     (min_thickness 0.254)
-    (fill yes (arc_segments 16) (thermal_gap 0.508) (thermal_bridge_width 0.508))
+    (fill (arc_segments 16) (thermal_gap 0.508) (thermal_bridge_width 0.508))
     (polygon
       (pts
@@
     (connect_pads (clearance 0.508))
     (min_thickness 0.254)
-    (fill yes (arc_segments 16) (thermal_gap 0.508) (thermal_bridge_width 0.508))
+    (fill (arc_segments 16) (thermal_gap 0.508) (thermal_bridge_width 0.508))
     (polygon
       (pts
@@
     (connect_pads (clearance 0.508))
     (min_thickness 0.254)
-    (fill yes (arc_segments 16) (thermal_gap 0.508) (thermal_bridge_width 0.508))
+    (fill (arc_segments 16) (thermal_gap 0.508) (thermal_bridge_width 0.508))
     (polygon
       (pts
@@
     (connect_pads (clearance 0.508))
     (min_thickness 0.254)
-    (fill yes (arc_segments 16) (thermal_gap 0.508) (thermal_bridge_width 0.508))
+    (fill (arc_segments 16) (thermal_gap 0.508) (thermal_bridge_width 0.508))
     (polygon
       (pts
-        (xy 67.0375 69.9325) (xy 67.0375 79.9325) (xy 56.0375 79.9325) (xy 56.0375 69.9325)
+        (xy 67.0375 69.9325) (xy 67.0375 79.9325) (xy 56.0375 79.9325) (xy 56.0375 71.4325) (xy 57.5375 69.9325)
       )
     )
