File: mpio_projekty/resetUSBv4.98com2/resetUSB.sch (KiCad schematic (older format))
At the start: 68 parts, among them J1 USBB-G-SMD, J10 FC68391, J2 TUEA4F2SOBHT, J3 Conn_02x05, J4 SWD_4pin, J5 DE09-SL-24, J6 Conn_02x05, J7 AC3MAH-AU-PRE, J8 Mini-Fit Jr; 4,2mm, J9 FC68391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

Commit message: pisakUS
Connections:
- net USB_M renamed USB_DM
- net USB_P renamed USB_DP
Changed lines of the file:
@@
 	2250 3500 2300 3500
 Text Label 2300 3500 0    60   ~ 0
-USB_M
+USB_DM
 Text Label 2300 3600 0    60   ~ 0
-USB_P
+USB_DP
 $Comp
 L mpio_lib:AO4616 U6
@@
 SWDIO
 Text Label 10700 2400 0    60   ~ 0
-USB_P
+USB_DP
 Text Label 10700 2300 0    60   ~ 0
-USB_M
+USB_DM
 Wire Wire Line
 	10700 2300 10650 2300
