File: mpio_projekty/pisakUS/pisakUS.kicad_pcb (KiCad board)
At the start: 2 copper layers, 12.7 x 21.1 mm, 7 parts, among them J1 Audio-Jack-4, J2 Conn_01x01, J3 Conn_01x01, U1 switch_no_nc_3pin

Commit message: pisakUS
Parts:
- moved R1 5.84 mm to (172.7, 84.3)
- moved R2 5.84 mm to (163.6, 84.3)
Routing:
- net GND: track 23.6 -> 35.9 mm
- net +3V3: track 17.5 -> 7.79 mm
- net Net-(D1-Pad2): track 20.2 -> 14.7 mm
Other:
- board size 12.7 x 21.1 mm -> 12.7 x 18.7 mm
