File: mpio_projekty/resetUSBv4.99/resetUSB.kicad_pcb (KiCad board)
At the start: 2 copper layers, 45 x 165 mm, 69 parts, among them J1 USBB-G-SMD, J10 FC68391, J2 TUEA4F2SOBHT, J3 Conn_02x05, J4 SWD_4pin, J5 DE09-SL-24, J6 Conn_02x05, J7 AC3MAH-AU-PRE, J8 Mini-Fit Jr; 4,2mm, J9 FC68391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

Commit message: KnoockerV2
Parts:
- removed R6: 10K, Resistors_SMD:R_0603
- removed REF**: SK48-50-SA-3, mpio:SK48-50-SA-3
- MK1: value RAD-A5723/60 -> SK48-50-SA-3; footprint mpio:RAD-A5723-60 -> mpio:SK48-50-SA-3
- moved MK1 27.5 mm to (81.0, 172.4)
- moved C9 7.49 mm to (66.8, 133.7), turned to 0 degrees
Routing:
- net Net-(LS1-Pad2): track 109.2 -> 22.2 mm
- net GND: track 44.6 -> 85.5 mm, vias 25 -> 26
- net +12V: track 257.4 -> 297.7 mm
- net Net-(J9-Pad1): track 50.8 -> 72.5 mm
- net Net-(D10-Pad1): track 13.8 -> 33.6 mm
- net Net-(J10-Pad1): track 54.4 -> 73.4 mm
- net Net-(Q1-Pad1): track 0.00 -> 11.0 mm
- net Net-(Q2-Pad1): track 0.00 -> 9.41 mm
- net Net-(LS2-Pad1): track 19.8 -> 20.4 mm
Other:
- board text added: "+USB+"
- board text added: "-USB-"
- board text added: "Knoocker_V2 marekp18@ gmail.com"
- board text removed: "Knoocker resetUSBv4 marekp18@ gmail.com"
- board text removed: "USB"
