File: mpio_projekty/resetUSBv4.99/resetUSB.sch (KiCad schematic (older format))
At the start: 68 parts, among them J1 USBB-G-SMD, J10 FC68391, J2 TUEA4F2SOBHT, J3 Conn_02x05, J4 SWD_4pin, J5 DE09-SL-24, J6 Conn_02x05, J7 AC3MAH-AU-PRE, J8 Mini-Fit Jr; 4,2mm, J9 FC68391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

Commit message: KnoockerV2
Parts:
- removed R6: 10K, Resistors_SMD:R_0603, symbol device:R
- MK1: value RAD-A5723/60 -> SK48-50-SA-3; footprint mpio:RAD-A5723-60 -> mpio:SK48-50-SA-3
Changed lines of the file:
@@
 P 4300 6500
 F 0 "MK1" H 4400 6546 50  0000 L CNN
-F 1 "RAD-A5723/60" H 4400 6455 50  0000 L CNN
-F 2 "mpio:RAD-A5723-60" H 4300 6500 50  0001 C CNN
+F 1 "SK48-50-SA-3" H 4400 6455 50  0000 L CNN
+F 2 "mpio:SK48-50-SA-3" H 4300 6500 50  0001 C CNN
 F 3 "" H 4300 6500 50  0001 C CNN
 	1    4300 6500
@@
 Text Label 6150 5350 2    60   ~ 0
 TX
-Text Label 5900 5550 2    60   ~ 0
+Text Label 6150 5550 2    60   ~ 0
 RX
 $Comp
@@
 Wire Wire Line
 	6150 5350 6200 5350
-Wire Wire Line
-	5900 5550 5950 5550
 NoConn ~ 6200 5850
 NoConn ~ 6200 5750
@@
 Wire Wire Line
 	10650 1500 10700 1500
-$Comp
-L device:R R6
-U 1 1 5B420233
-P 5950 5350
-F 0 "R6" V 6030 5350 50  0000 C CNN
-F 1 "10K" V 5950 5350 50  0000 C CNN
-F 2 "Resistors_SMD:R_0603" V 5880 5350 50  0001 C CNN
-F 3 "" H 5950 5350 50  0001 C CNN
-	1    5950 5350
-	-1   0    0    -1
-$EndComp
-Wire Wire Line
-	5950 5500 5950 5550
-Connection ~ 5950 5550
-Wire Wire Line
-	5950 5550 6200 5550
-$Comp
-L power:+3V3 #PWR0114
-U 1 1 5B44AFCE
-P 5950 5150
-F 0 "#PWR0114" H 5950 5000 50  0001 C CNN
-F 1 "+3V3" H 5950 5290 50  0000 C CNN
-F 2 "" H 5950 5150 50  0001 C CNN
-F 3 "" H 5950 5150 50  0001 C CNN
-	1    5950 5150
-	1    0    0    -1
-$EndComp
-Wire Wire Line
-	5950 5150 5950 5200
 $Comp
 L power:GND #PWR0115
@@
 Wire Wire Line
 	1500 3700 1750 3700
+Wire Wire Line
+	6150 5550 6200 5550
 $EndSCHEMATC
